File: LEDDriver.kicad_sch (KiCad schematic)
At the start: 44 parts

Commit message: completed schematics
Parts:
- removed D? (x6): LED_RGB_3, symbol Device:LED_RGB_3
- removed D? (x2): LED_RGB_5, symbol Device:LED_RGB_5
- removed D? (x2): LED_RGB_1, symbol Device:LED_RGB_1
- removed D?: LED_RGB_2, symbol Device:LED_RGB_2
- removed D?: LED_RGB_4, symbol Device:LED_RGB_4
- added D28, D29, D30, D31, D32: LED_RGB_2, AnalogueWallClockMirrorFootprintsLibrary:APF3236SEEZGQBDC_Hole, symbol Device:LED_RGB_2
- added D48, D49, D50, D51, D52, D53: LED_BGRA_1, LED_SMD:QBLP677R-RGB, symbol Device:LED_BGRA
- added D54, D55, D56, D57, D58, D59: LED_RABG, LED_SMD:XZMDKCBDDG45S-9, symbol Device:LED_RABG
- added D60, D61, D62, D63, D64, D65: LED_ABRG, LED_SMD:156120M173000, symbol Device:LED_ABRG
- D13, D14, D15, D16, D17: renamed from D?; footprint (none) -> AnalogueWallClockMirrorFootprintsLibrary:19-337C_RSBHGHC-A88_4T_Cutout
- D18, D19, D20, D21, D22: renamed from D?; footprint (none) -> AnalogueWallClockMirrorFootprintsLibrary:19-337C_RSBHGHC-A88_4T_Hole
- D23, D24, D25, D26, D27: renamed from D?; footprint (none) -> AnalogueWallClockMirrorFootprintsLibrary:APF3236SEEZGQBDC_Cutout
- D33, D34, D35, D36, D37: renamed from D?; footprint (none) -> AnalogueWallClockMirrorFootprintsLibrary:CLP6C-FKB-CK1P1G1BB7R3R3_Hole
- D38, D39, D40, D41, D42: renamed from D?; footprint (none) -> AnalogueWallClockMirrorFootprintsLibrary:SMLVN6RGB1W1‎_Cutout
- D43, D44, D45, D46, D47: renamed from D?; footprint (none) -> AnalogueWallClockMirrorFootprintsLibrary:SMLVN6RGB1W1‎_Hole
- U6: renamed from U?; footprint (none) -> Package_DFN_QFN:QFN-76_EP_9.1x9.1_Pitch0.4mm
Connections:
- net B3: now also D28.6 (BA), D29.6 (BA), D30.6 (BA), D31.6 (BA), D32.6 (BA)
- net G3: now also D28.5 (GA), D29.5 (GA), D30.5 (GA), D31.5 (GA), D32.5 (GA)
- net L0: now also D28.1 (RK), D28.2 (GK), D28.3 (BK), D48.3 (RK), D54.1 (RK), D60.3 (RK)
- net L1: now also D29.1 (RK), D29.2 (GK), D29.3 (BK), D49.3 (RK), D55.1 (RK), D61.3 (RK)
- net L2: now also D30.1 (RK), D30.2 (GK), D30.3 (BK), D50.2 (GK), D56.4 (GK), D62.4 (GK)
- net L3: now also D31.1 (RK), D31.2 (GK), D31.3 (BK), D51.2 (GK), D57.4 (GK), D63.4 (GK)
- net L4: now also D32.1 (RK), D32.2 (GK), D32.3 (BK), D52.1 (BK), D58.3 (BK), D64.2 (BK)
- net L5: now also D53.1 (BK), D59.3 (BK), D65.2 (BK)
- net R3: now also D28.4 (RA), D29.4 (RA), D30.4 (RA), D31.4 (RA), D32.4 (RA)
- net R7: now reaches U6.27 (R7)
- net R7: now also D48.4 (A), D49.4 (A)
- net G7: now reaches U6.28 (G7)
- net G7: now also D50.4 (A), D51.4 (A)
- net B7: now reaches U6.29 (B7)
- net B7: now also D52.4 (A), D53.4 (A)
- net B8: now reaches U6.30 (B8)
- net B8: now also D58.2 (A), D59.2 (A)
- net G8: now reaches U6.31 (G8)
- net G8: now also D56.2 (A), D57.2 (A)
- net R8: now reaches U6.32 (R8)
- net R8: now also D54.2 (A), D55.2 (A)
- net B9: now reaches U6.33 (B9)
- net B9: now also D64.1 (A), D65.1 (A)
- net G9: now reaches U6.34 (G9)
- net G9: now also D62.1 (A), D63.1 (A)
- net R9: now reaches U6.35 (R9)
- net R9: now also D60.1 (A), D61.1 (A)
- no-connect marks 37 -> 64
