File: PowCon.kicad_sch (KiCad schematic)
At the start: 63 parts

Commit message: completed schematics
Parts:
- added D11, D12: LED_RGB_3, LED_SMD:APTF3216QBDZGSURKC, symbol Device:LED_RGB_2
- added Q1, Q2, Q3: NX7002BKWX, Package_TO_SOT_SMD:SOT-323_SC-70_Handsoldering, symbol Device:Q_NMOS_GSD
- added R10, R8, R9: 1k, Resistor_SMD:R_0603_1608Metric_Pad0.98x0.95mm_HandSolder, symbol Device:R
- added R13, R15, R16, R17, R18, R23, R24, R25, R5, R6, R7: 22R, Resistor_SMD:R_0603_1608Metric_Pad0.98x0.95mm_HandSolder, symbol Device:R
- added R28, R31: 232R, Resistor_SMD:R_0603_1608Metric_Pad0.98x0.95mm_HandSolder, symbol Device:R
- added R29, R32: 309R, Resistor_SMD:R_0603_1608Metric_Pad0.98x0.95mm_HandSolder, symbol Device:R
- added R30, R33: 590R, Resistor_SMD:R_0603_1608Metric_Pad0.98x0.95mm_HandSolder, symbol Device:R
- JP1: renamed from JP?; footprint (none) -> Jumper:SolderJumper-2_P1.3mm_Open_TrianglePad1.0x1.5mm; now left out of the parts list
- U6: renamed from U?; footprint (none) -> Package_DFN_QFN:QFN-76_EP_9.1x9.1_Pitch0.4mm
- gave numbers to parts that had none: 61
Connections:
- net +5V: now also R30.2, R33.2
- net I2C_SCL: now also R15.2; no longer R12.2, U1.24 (IO2)
- net I2C_SDA: now also R13.2; no longer R4.2, U1.23 (IO15)
- net SPI_CLK: now also R23.2; no longer R20.2, U1.30 (IO18)
- net SPI_SDOUT: now also R25.2; no longer R22.2, U1.37 (IO23)
- net SPI_SIN: now also R24.2; no longer R21.2, U1.31 (IO19)
- net VDD: now also R28.2, R31.2
- net VDD_U/~{D}: now also R17.2; no longer U1.29 (IO5)
- net VDD_~{CS}: now also R18.2; no longer U1.14 (IO12)
- net VDD_~{INC}: now also R16.2; no longer U1.26 (IO4)
- net VEE: now also R29.2, R32.2
- net VEE_U/~{D}: now also R6.2; no longer U1.11 (IO26)
- net VEE_~{CS}: now also R7.2; no longer U1.12 (IO27)
- net VEE_~{INC}: now also R5.2; no longer U1.10 (IO25)
- net at U1.36 (IO22): now also R10.1
- net at U1.8 (IO32): now also R8.1
- net at U1.9 (IO33): now also R9.1
- removed net GND: C1.2, C10.2, C11.2, C12.2, C13.2, C14.2, C15.2, C16.2, C17.2, C18.2, C19.2, C2.2, C20.2, C21.2, C22.2, C3.2, C4.2, C5.2, C6.2, C7.2, C8.2, C9.2, D1.2 (A2), D10.2 (A2), D2.2 (A2), D3.2 (A2), D4.2 (A2), D5.2 (A2), D6.2 (A2), D7.2 (A2), D8.2 (A2), D9.2 (A2), J1.A12 (GND), J1.B12 (GND), J2.4 (GND), JP1.2 (B), R2.2, R27.1, R3.2, R37.1, R38.1, U1.1 (GND), U1.15 (GND), U1.38 (GND), U1.39 (GND), U2.2 (GND), U3.4 (GND), U3.6 (RL), U4.11 (GND), U4.3 (GND), U4.7 (GND), U5.3 (GND), U6.7 (GND), U6.77 (TPAD), U7.4 (GND), U7.6 (RL), U8.11 (GND), U8.3 (GND), U8.7 (GND)
- new net: R13.1, R4.2, U1.23 (IO15)
- new net: Q1.1 (G), R10.2
- new net: D3.2 (A2), D5.2 (A2), R2.2, R3.2
- new net: D11.5 (GA), R29.1
- new net: R21.2, R24.1, U1.31 (IO19)
- new net: Q2.1 (G), R8.2
- new net: JP1.2 (B), R27.1, U3.6 (RL)
- new net: C4.2, C6.2, U2.2 (GND)
- new net: D10.2 (A2), D6.2 (A2), D8.2 (A2)
- new net: D7.2 (A2), D9.2 (A2)
- new net: R16.1, U1.26 (IO4)
- new net: R17.1, U1.29 (IO5)
- new net: C12.2, C14.2, C17.2
- new net: R22.2, R25.1, U1.37 (IO23)
- new net: R5.1, U1.10 (IO25)
- new net: C20.2, C21.2
- new net: R20.2, R23.1, U1.30 (IO18)
- new net: D11.4 (RA), R28.1
- new net: D2.2 (A2), D4.2 (A2)
- new net: R12.2, R15.1, U1.24 (IO2)
- new net: D12.4 (RA), R31.1
- new net: U8.11 (GND), U8.3 (GND), U8.7 (GND)
- new net: R38.1, U7.6 (RL)
- new net: C5.2, C7.2
- new net: C2.2, C3.2
- new net: C16.2, C18.2, C19.2, C22.2
- new net: C1.2, J2.4 (GND)
- new net: D12.6 (BA), R33.1
- new net: R6.1, U1.11 (IO26)
- new net: U6.7 (GND), U6.77 (TPAD)
- new net: D11.1 (RK), Q1.3 (D)
- new net: D11.2 (GK), Q2.3 (D)
- new net: D11.3 (BK), Q3.3 (D)
- new net: D11.6 (BA), R30.1
- new net: C10.2, C11.2, U5.3 (GND)
- new net: D1.2 (A2), J1.A12 (GND), J1.B12 (GND)
- new net: Q3.1 (G), R9.2
- new net: U4.11 (GND), U4.3 (GND), U4.7 (GND)
- new net: C13.2, C15.2
- new net: D12.5 (GA), R32.1
- new net: D12.1 (RK), D12.2 (GK), D12.3 (BK)
- new net: C8.2, C9.2
- new net: U1.1 (GND), U1.15 (GND), U1.38 (GND), U1.39 (GND)
- new net: R7.1, U1.12 (IO27)
- new net: R18.1, U1.14 (IO12)
- no-connect marks 2 -> 17
Other:
- moved on the sheet: C12, C14, C16, C17, C18, C19, C22, R11, R20, R21, R22, R37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
