File: AnalogueWallClock.kicad_sch (KiCad schematic)
At the start: 8 parts

Commit message: completed schematics
Parts:
- added S1: M3 Screw, symbol Mechanical:MountingHole
- added S2, S3, S4, S5, S6: M3 Thumb Screw, symbol Mechanical:MountingHole
- FID1, FID2, FID3: renamed from FID?; footprint (none) -> Fiducial:Fiducial_0.75mm_Mask1.5mm
- H1, H2, H3, H4, H5: renamed from H?; footprint (none) -> MountingHole:MountingHole_3.5mm

Commit message: test pcb complete
Parts:
- removed H1, H2, H3, H4, H5: MountingHole, MountingHole:MountingHole_3.5mm, symbol Mechanical:MountingHole
- removed S1: M3 Screw, symbol Mechanical:MountingHole
- removed S2, S3, S4, S5, S6: M3 Thumb Screw, symbol Mechanical:MountingHole
- added D1: LED_RGB_1, AnalogueWallClockMirrorFootprintsLibrary:19-337C_RSBHGHC-A88_4T_Cutout, symbol Device:LED_RGB_1
- added D10: LED_ABRG, LED_SMD:156120M173000, symbol Device:LED_ABRG
- added D2: LED_RGB_1, AnalogueWallClockMirrorFootprintsLibrary:19-337C_RSBHGHC-A88_4T_Hole, symbol Device:LED_RGB_1
- added D3: LED_RGB_2, AnalogueWallClockMirrorFootprintsLibrary:APF3236SEEZGQBDC_Cutout, symbol Device:LED_RGB_2
- added D4: LED_RGB_2, AnalogueWallClockMirrorFootprintsLibrary:APF3236SEEZGQBDC_Hole, symbol Device:LED_RGB_2
- added D5: LED_RGB_4, AnalogueWallClockMirrorFootprintsLibrary:CLP6C-FKB-CK1P1G1BB7R3R3_Hole, symbol Device:LED_RGB_4
- added D6: LED_RGB_5, AnalogueWallClockMirrorFootprintsLibrary:SMLVN6RGB1W1‎_Cutout, symbol Device:LED_RGB_5
- added D7: LED_RGB_5, AnalogueWallClockMirrorFootprintsLibrary:SMLVN6RGB1W1‎_Hole, symbol Device:LED_RGB_5
- added D8: LED_BGRA_1, LED_SMD:QBLP677R-RGB, symbol Device:LED_BGRA
- added D9: LED_RABG, LED_SMD:XZMDKCBDDG45S-9, symbol Device:LED_RABG
- added J1: USB_C, Connector_USB:USB-C-PowerOnly, symbol Connector:USB_C_Receptacle_USB2.0_1
- added R1, R2: 5.1k, Resistor_SMD:R_0603_1608Metric_Pad0.98x0.95mm_HandSolder, symbol Device:R
- added R10, R13, R16, R19, R22, R25, R28, R31, R4, R7: 191R, Resistor_SMD:R_0603_1608Metric_Pad0.98x0.95mm_HandSolder, symbol Device:R
- added R11, R14, R17, R20, R23, R26, R29, R32, R5, R8: 412R, Resistor_SMD:R_0603_1608Metric_Pad0.98x0.95mm_HandSolder, symbol Device:R
- added R12, R15, R18, R21, R24, R27, R3, R30, R6, R9: 357R, Resistor_SMD:R_0603_1608Metric_Pad0.98x0.95mm_HandSolder, symbol Device:R
Connections:
- new net: D9.3 (BK), R29.1
- new net: D10.2 (BK), R32.1
- new net: D10.3 (RK), R30.1
- new net: D10.4 (GK), R31.1
- new net: D4.2 (GK), R13.1
- new net: D3.3 (BK), R11.1
- new net: D9.4 (GK), R28.1
- new net: D2.3 (RK), R6.1
- new net: D9.1 (RK), R27.1
- new net: J1.A5 (CC1), R2.1
- new net: J1.B5 (CC2), R1.1
- new net: D7.5 (RK), R21.1
- new net: D2.5 (BK), R8.1
- new net: D5.6 (RK), R15.1
- new net: D1.1 (GK), R4.1
- new net: D1.3 (RK), R3.1
- new net: D1.5 (BK), R5.1
- new net: D7.4 (GK), R22.1
- new net: D7.6 (BK), R23.1
- new net: D8.2 (GK), R25.1
- new net: D4.3 (BK), R14.1
- new net: D5.5 (GK), R16.1
- new net: D4.1 (RK), R12.1
- new net: D5.4 (BK), R17.1
- new net: D6.6 (BK), R20.1
- new net: D6.5 (RK), R18.1
- new net: D2.1 (GK), R7.1
- new net: D8.3 (RK), R24.1
- new net: D3.1 (RK), R9.1
- new net: D3.2 (GK), R10.1
- new net: D6.4 (GK), R19.1
- new net: D8.1 (BK), R26.1
- new net +5V: D1.2 (GA), D1.4 (RA), D1.6 (BA), D10.1 (A), D2.2 (GA), D2.4 (RA), D2.6 (BA), D3.4 (RA), D3.5 (GA), D3.6 (BA), D4.4 (RA), D4.5 (GA), D4.6 (BA), D5.1 (RA), D5.2 (GA), D5.3 (BA), D6.1 (BA), D6.2 (RA), D6.3 (GA), D7.1 (BA), D7.2 (RA), D7.3 (GA), D8.4 (A), D9.2 (A), J1.A9 (VBUS), J1.B9 (VBUS)
- new net GND: J1.A12 (GND), J1.B12 (GND), R1.2, R10.2, R11.2, R12.2, R13.2, R14.2, R15.2, R16.2, R17.2, R18.2, R19.2, R2.2, R20.2, R21.2, R22.2, R23.2, R24.2, R25.2, R26.2, R27.2, R28.2, R29.2, R3.2, R30.2, R31.2, R32.2, R4.2, R5.2, R6.2, R7.2, R8.2, R9.2
- no-connect marks 0 -> 1
Other:
- removed sheet LED Driver
- removed sheet Power & Control
